File: 2 - Board Files/2 - PowerDistribution/MotorDrive.kicad_sch (KiCad schematic)
At the start: 0 parts

Commit message: Motor drive initial work
Parts:
- added C601, C602, C603, C604, C605, C606, C607, C608, C609, C610, C611, C612, C613, C614, C615, C616, C617, C618, C619, C620, C621, C622, C623, C624: 0u1, Capacitor_SMD:C_0402_1005Metric, symbol Device:C_Small
- added Q601, Q602, Q603, Q604, Q605, Q606, Q607, Q608, Q609, Q610, Q611, Q612, Q613, Q614, Q615, Q616, Q617, Q618, Q619, Q620, Q621, Q622, Q623, Q624: Q_NMOS_GDS, Package_TO_SOT_SMD:Infineon_PG-HSOF-8-1, symbol Device:Q_NMOS_GDS
- added R601, R602, R603, R604, R606, R607, R608, R609, R611, R612, R613, R614, R615, R616, R617, R618: 4k7, Resistor_SMD:R_0402_1005Metric, symbol Device:R_Small_US
- added R605, R610, R619, R620: 1m, 3W, Resistor_SMD:R_1206_3216Metric, symbol Device:R_Small_US
- added U601, U602, U603, U604: BD63003MUV, Package_DFN_QFN:QFN-32-1EP_5x5mm_P0.5mm_EP3.65x3.65mm, symbol QuadrotorLib:BD63003MUV
Connections:
- new net: Q624.1 (G), U604.14 (WL)
- new net: Q622.3 (S), Q624.2 (D), U604.15 (W)
- new net: Q616.3 (S), Q620.3 (S), Q624.3 (S), R620.2, U604.17 (RCL)
- new net: Q613.1 (G), U603.10 (UH)
- new net: Q613.3 (S), Q615.2 (D), U603.9 (U)
- new net: Q615.1 (G), U603.8 (UL)
- new net: Q615.3 (S), Q619.3 (S), Q623.3 (S), R619.2, U603.17 (RCL)
- new net: Q605.1 (G), U601.16 (WH)
- new net: Q605.3 (S), Q606.2 (D), U601.15 (W)
- new net: R613.2, U603.1 (FG)
- new net: Q617.1 (G), U603.11 (VH)
- new net: Q617.3 (S), Q619.2 (D), U603.12 (V)
- new net: Q619.1 (G), U603.13 (VL)
- new net: Q623.1 (G), U603.14 (WL)
- new net: Q621.3 (S), Q623.2 (D), U603.15 (W)
- new net: Q621.1 (G), U603.16 (WH)
- new net: R612.1, U603.27 (SEL2)
- new net: C621.1, U603.29 (CP1)
- new net: C621.2, U603.30 (CP2)
- new net: C620.2, U603.31 (VG)
- new net: R617.1, U603.5 (IREF)
- new net: R611.1, U603.6 (SEL1)
- new net: C612.1, U602.29 (CP1)
- new net: C612.2, U602.30 (CP2)
- new net: Q601.1 (G), U601.10 (UH)
- new net: Q601.3 (S), Q602.2 (D), U601.9 (U)
- new net: R615.1, U604.27 (SEL2)
- new net: Q610.1 (G), U602.13 (VL)
- new net: Q609.3 (S), Q610.2 (D), U602.12 (V)
- new net: Q608.3 (S), Q610.3 (S), Q612.3 (S), R610.2, U602.17 (RCL)
- new net: R603.2, U601.1 (FG)
- new net: Q603.1 (G), U601.11 (VH)
- new net: Q603.3 (S), Q604.2 (D), U601.12 (V)
- new net: Q604.1 (G), U601.13 (VL)
- new net: Q606.1 (G), U601.14 (WL)
- new net: Q602.3 (S), Q604.3 (S), Q606.3 (S), R605.2, U601.17 (RCL)
- new net: R602.1, U601.27 (SEL2)
- new net: C603.1, U601.29 (CP1)
- new net: C603.2, U601.30 (CP2)
- new net: C602.2, U601.31 (VG)
- new net: R604.1, U601.5 (IREF)
- new net: R601.1, U601.6 (SEL1)
- new net: Q602.1 (G), U601.8 (UL)
- new net: Q611.1 (G), U602.16 (WH)
- new net: Q611.3 (S), Q612.2 (D), U602.15 (W)
- new net: Q618.1 (G), U604.11 (VH)
- new net: Q618.3 (S), Q620.2 (D), U604.12 (V)
- new net: Q608.1 (G), U602.8 (UL)
- new net: Q607.3 (S), Q608.2 (D), U602.9 (U)
- new net: Q612.1 (G), U602.14 (WL)
- new net: Q620.1 (G), U604.13 (VL)
- new net: R608.2, U602.1 (FG)
- new net: Q607.1 (G), U602.10 (UH)
- new net: Q609.1 (G), U602.11 (VH)
- new net: R607.1, U602.27 (SEL2)
- new net: C611.2, U602.31 (VG)
- new net: R609.1, U602.5 (IREF)
- new net: R606.1, U602.6 (SEL1)
- new net: R618.1, U604.5 (IREF)
- new net: Q622.1 (G), U604.16 (WH)
- new net: Q616.1 (G), U604.8 (UL)
- new net: Q614.3 (S), Q616.2 (D), U604.9 (U)
- new net: C624.1, U604.29 (CP1)
- new net: C624.2, U604.30 (CP2)
- new net: R616.2, U604.1 (FG)
- new net: Q614.1 (G), U604.10 (UH)
- new net: C623.2, U604.31 (VG)
- new net: R614.1, U604.6 (SEL1)
- new net +BATT: C601.1, C602.1, C604.1, C605.1, C606.1, C607.1, C608.1, C609.1, C610.1, C611.1, C613.1, C614.1, C615.1, C616.1, C617.1, C618.1, C619.1, C620.1, C622.1, C623.1, Q601.2 (D), Q603.2 (D), Q605.2 (D), Q607.2 (D), Q609.2 (D), Q611.2 (D), Q613.2 (D), Q614.2 (D), Q617.2 (D), Q618.2 (D), Q621.2 (D), Q622.2 (D), R603.1, R608.1, R613.1, R616.1, U601.32 (VCC), U601.4 (BRKB), U602.32 (VCC), U602.4 (BRKB), U603.32 (VCC), U603.4 (BRKB), U604.32 (VCC), U604.4 (BRKB)
- new net GND: C601.2, C604.2, C605.2, C606.2, C607.2, C608.2, C609.2, C610.2, C613.2, C614.2, C615.2, C616.2, C617.2, C618.2, C619.2, C622.2, R601.2, R602.2, R604.2, R605.1, R606.2, R607.2, R609.2, R610.1, R611.2, R612.2, R614.2, R615.2, R617.2, R618.2, R619.1, R620.1, U601.18 (RCLS), U601.28 (TEST), U601.3 (CW), U601.33 (GND_EP), U601.7 (GND), U602.18 (RCLS), U602.28 (TEST), U602.3 (CW), U602.33 (GND_EP), U602.7 (GND), U603.18 (RCLS), U603.28 (TEST), U603.3 (CW), U603.33 (GND_EP), U603.7 (GND), U604.18 (RCLS), U604.28 (TEST), U604.3 (CW), U604.33 (GND_EP), U604.7 (GND)
- new net MOTOR1_PWM: U601.2 (PWMB), U602.2 (PWMB), U603.2 (PWMB), U604.2 (PWMB)
- no-connect marks 0 -> 32
Other:
- note added: "Add filteration?"
- note added: "CW has internal PUR"
- note added: "Pull high to disable braking"

Commit message: MOSFETs changed
Parts:
- added J601, J602, J603, J604: Conn_01x03_Female, QuadrotorFootprints:MotorOutputPads, symbol Connector:Conn_01x03_Female
- Q601, Q602, Q603, Q604, Q605, Q606: footprint Package_TO_SOT_SMD:Infineon_PG-HSOF-8-1 -> QuadrotorFootprints:8-PowerVDFN; PN (none) -> RQ3E070BNTB
- Q607, Q608, Q609, Q610, Q611, Q612, Q613, Q614, Q615, Q616, Q617, Q618, Q619, Q620, Q621, Q622, Q623, Q624: footprint Package_TO_SOT_SMD:Infineon_PG-HSOF-8-1 -> QuadrotorFootprints:8-PowerVDFN
Connections:
- net GND: no longer U602.3 (CW), U604.3 (CW)
- net MOTOR1_PWM: no longer U602.2 (PWMB), U603.2 (PWMB), U604.2 (PWMB)
- net at Q622.3 (S), Q624.2 (D), U604.15 (W): now also J604.3 (Pin_3)
- net at Q613.3 (S), Q615.2 (D), U603.9 (U): now also J603.1 (Pin_1)
- net at Q605.3 (S), Q606.2 (D), U601.15 (W): now also J601.3 (Pin_3)
- net at Q617.3 (S), Q619.2 (D), U603.12 (V): now also J603.2 (Pin_2)
- net at Q621.3 (S), Q623.2 (D), U603.15 (W): now also J603.3 (Pin_3)
- net at Q601.3 (S), Q602.2 (D), U601.9 (U): now also J601.1 (Pin_1)
- net at Q609.3 (S), Q610.2 (D), U602.12 (V): now also J602.2 (Pin_2)
- net at Q603.3 (S), Q604.2 (D), U601.12 (V): now also J601.2 (Pin_2)
- net at Q611.3 (S), Q612.2 (D), U602.15 (W): now also J602.3 (Pin_3)
- net at Q618.3 (S), Q620.2 (D), U604.12 (V): now also J604.2 (Pin_2)
- net at Q607.3 (S), Q608.2 (D), U602.9 (U): now also J602.1 (Pin_1)
- net at Q614.3 (S), Q616.2 (D), U604.9 (U): now also J604.1 (Pin_1)
- new net MOTOR2_PWM: U602.2 (PWMB)
- new net MOTOR3_PWM: U603.2 (PWMB)
- new net MOTOR4_PWM: U604.2 (PWMB)
- no-connect marks 32 -> 34
Other:
- note added: "ALL FETS P/N: RQ3E070BNTB"
- moved on the sheet: C613, C614, C615, C616, C617, C618, C619, C620, C621, C622, C623, C624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
